File: microbyte-rp2040/microbyte-rp2040.sch (KiCad schematic (older format))
At the start: 54 parts, among them J1 BATT_CON, J2 TF-15X15, J3 USB_CONN, J4 HEADERS, Q1 AO3401A, SW1 BOOT, SW2 RESET, U1 AP2112K-3.3, U2 MCP73831-2-OT, U3 W25QXX128MBIT, U4 RP2040, Y1 12MHz

Commit message: microbyte-rp2040-v1.1
Parts:
- removed C3: 4u7, Capacitor_SMD:C_0603_1608Metric, symbol Device:C_Small
- removed D2: YELLOW, LED_SMD:LED_0603_1608Metric, symbol Device:LED_Small
- removed R3: 2k, Resistor_SMD:R_0603_1608Metric, symbol Device:R_Small
- removed R4: 1k, Resistor_SMD:R_0402_1005Metric, symbol Device:R_Small
- removed U2: MCP73831-2-OT, Package_TO_SOT_SMD:SOT-23-5, symbol Battery_Management:MCP73831-2-OT
- added JP1: 3V3_JMP, Jumper:SolderJumper-2_P1.3mm_Open_RoundedPad1.0x1.5mm, symbol Jumper:SolderJumper_2_Open
- added JP2: 5V_JMP, Jumper:SolderJumper-2_P1.3mm_Open_RoundedPad1.0x1.5mm, symbol Jumper:SolderJumper_2_Open
- SW1, SW2: footprint Button_Switch_SMD:Panasonic_EVQPUL_EVQPUC -> Button_Switch_SMD:SW_SPST_TL3342; LCSC C79175 -> C318889
- renumbered C4 to C3, D4 to D2, D5 to D3, D6 to D4
Connections:
- net +3.3VA: now also J4.7 (Pin_7); no longer J4.6 (Pin_6)
- net +3V3: now also J4.1 (Pin_1), J4.17 (Pin_17), JP1.2 (B); no longer C2.1, J4.4 (Pin_4), U1.5 (VOUT)
- net +5V: now also J4.2 (Pin_2), J4.4 (Pin_4), JP2.2 (B); no longer J3.A4 (VBUS), J3.A9 (VBUS), J3.B4 (VBUS), J3.B9 (VBUS), J4.5 (Pin_5)
- net +BATT: now also J4.37 (Pin_37); no longer J4.1 (Pin_1)
- net ADC0: now also J4.24 (Pin_24); no longer J4.10 (Pin_10)
- net ADC1: now also J4.22 (Pin_22); no longer J4.12 (Pin_12)
- net ADC2: now also J4.18 (Pin_18); no longer J4.14 (Pin_14)
- net GND: now also J4.14 (Pin_14), J4.20 (Pin_20), J4.25 (Pin_25), J4.30 (Pin_30), J4.34 (Pin_34), J4.39 (Pin_39), J4.6 (Pin_6), J4.9 (Pin_9); no longer J4.24 (Pin_24), J4.8 (Pin_8)
- net GPIO16: now also J4.35 (Pin_35); no longer J4.7 (Pin_7)
- net GPIO17: now also J4.33 (Pin_33); no longer J4.9 (Pin_9)
- net GPIO18: now also J4.31 (Pin_31); no longer J4.11 (Pin_11)
- net GPIO19: now also J4.29 (Pin_29); no longer J4.13 (Pin_13)
- net GPIO20: now also J4.27 (Pin_27); no longer J4.15 (Pin_15)
- net GPIO21: now also J4.23 (Pin_23); no longer J4.17 (Pin_17)
- net GPIO22: now also J4.21 (Pin_21); no longer J4.19 (Pin_19)
- net GPIO23: now also J4.19 (Pin_19); no longer J4.21 (Pin_21)
- net GPIO24: now also J4.15 (Pin_15); no longer J4.23 (Pin_23)
- net GPIO25: now also J4.13 (Pin_13); no longer J4.25 (Pin_25)
- net GPIO5: now also J4.32 (Pin_32); no longer J4.36 (Pin_36)
- net I2C1_SCL: now also J4.5 (Pin_5); no longer J4.40 (Pin_40)
- net I2C1_SDA: now also J4.3 (Pin_3); no longer J4.38 (Pin_38)
- net RESET: no longer J4.2 (Pin_2)
- net SPI0_MISO: now also J4.40 (Pin_40); no longer J4.34 (Pin_34)
- net SPI0_MOSI: now also J4.38 (Pin_38); no longer J4.32 (Pin_32)
- net SPI0_SCK: now also J4.36 (Pin_36); no longer J4.30 (Pin_30)
- net SWDCK: now also J4.28 (Pin_28); no longer J4.22 (Pin_22)
- net SWDIO: now also J4.26 (Pin_26); no longer J4.20 (Pin_20)
- net UART0_RX: now also J4.10 (Pin_10); no longer J4.28 (Pin_28)
- net UART0_TX: now also J4.8 (Pin_8); no longer J4.26 (Pin_26)
- net EN: no longer names the net of R2.1, U1.3 (EN)
- net EN: no longer J4.3 (Pin_3)
- new net: C2.1, JP1.1 (A), U1.5 (VOUT)
- new net: J3.A4 (VBUS), J3.A9 (VBUS), J3.B4 (VBUS), J3.B9 (VBUS), JP2.1 (A)
- no-connect marks 11 -> 5
Other:
- note added: "Battery Connector"
- note removed: "+BATT should be a single-\ncell LiPo battery"
- note removed: "Charge current:\nI_CHG = 1000 / R_PROG\nR_PROG=2k : I_CHG=500mA"
- note removed: "Lithium-Polymer Battery Charger (1-cell)"
