File: microbyte-rp2040/microbyte-rp2040.kicad_pcb (KiCad board)
At the start: 4 copper layers, 65 x 30 mm, 56 parts, among them J1 BATT_CON, J2 TF-15X15, J3 USB_CONN, J4 HEADERS, Q1 AO3401A, SW1 BOOT, SW2 RESET, U1 AP2112K-3.3, U2 MCP73831-2-OT, U3 W25QXX128MBIT, U4 RP2040, Y1 12MHz

Commit message: microbyte-rp2040-v1.1
Parts:
- removed the C3 at (169.6, 100.3)
- removed the D2 at (179.0, 98.1)
- removed G***: LOGO, LOGO:microbyte_icon_3
- removed G***: LOGO, LOGO:microbyte_url_1
- removed R3: 2k, Resistor_SMD:R_0603_1608Metric
- removed R4: 1k, Resistor_SMD:R_0402_1005Metric
- removed U2: MCP73831-2-OT, Package_TO_SOT_SMD:SOT-23-5
- added JP1: 3V3_JMP, Jumper:SolderJumper-2_P1.3mm_Open_RoundedPad1.0x1.5mm, F.Cu at (145.0, 97.3)
- added JP2: 5V_JMP, Jumper:SolderJumper-2_P1.3mm_Open_RoundedPad1.0x1.5mm, F.Cu at (145.0, 94.4)
- SW1, SW2: footprint Button_Switch_SMD:Panasonic_EVQPUL_EVQPUC -> Button_Switch_SMD:SW_SPST_TL3342
- moved J1 14.0 mm to (170.0, 103.7), turned to 0 degrees
- moved D2 3.44 mm to (175.5, 101.0), turned to 90 degrees
- moved C3 2.22 mm to (170.0, 97.7)
- moved R6 1.75 mm to (176.9, 100.5), turned to 90 degrees
- moved SW2 1.51 mm to (119.6, 98.4), turned to 270 degrees
- moved SW1 1.50 mm to (119.6, 89.4), turned to 270 degrees
- moved R8 0.08 mm to (164.8, 102.6)
- renumbered C4 to C3, D4 to D2, D5 to D3, D6 to D4
Connections:
- C2 pad 1: +3V3 -> Net-(C2-Pad1)
- J3 pad A4: +5V -> Net-(J3-PadA4)
- J3 pad A9: +5V -> Net-(J3-PadA4)
- J3 pad B4: +5V -> Net-(J3-PadA4)
- J3 pad B9: +5V -> Net-(J3-PadA4)
- J4 pad 1: +BATT -> +3V3
- J4 pad 10: ADC0 -> UART0_RX
- J4 pad 11: GPIO18 -> Net-(J4-Pad11)
- J4 pad 12: ADC1 -> Net-(J4-Pad12)
- J4 pad 13: GPIO19 -> GPIO25
- J4 pad 14: ADC2 -> GND
- J4 pad 15: GPIO20 -> GPIO24
- J4 pad 17: GPIO21 -> +3V3
- J4 pad 18: Net-(J4-Pad18) -> ADC2
- J4 pad 19: GPIO22 -> GPIO23
- J4 pad 2: RESET -> +5V
- J4 pad 20: SWDIO -> GND
- J4 pad 21: GPIO23 -> GPIO22
- J4 pad 22: SWDCK -> ADC1
- J4 pad 23: GPIO24 -> GPIO21
- J4 pad 24: GND -> ADC0
- J4 pad 25: GPIO25 -> GND
- J4 pad 26: UART0_TX -> SWDIO
- J4 pad 27: Net-(J4-Pad27) -> GPIO20
- J4 pad 28: UART0_RX -> SWDCK
- J4 pad 29: Net-(J4-Pad29) -> GPIO19
- J4 pad 3: EN -> I2C1_SDA
- J4 pad 30: SPI0_SCK -> GND
- J4 pad 31: Net-(J4-Pad31) -> GPIO18
- J4 pad 32: SPI0_MOSI -> GPIO5
- J4 pad 33: Net-(J4-Pad33) -> GPIO17
- J4 pad 34: SPI0_MISO -> GND
- J4 pad 35: Net-(J4-Pad35) -> GPIO16
- J4 pad 36: GPIO5 -> SPI0_SCK
- J4 pad 37: Net-(J4-Pad37) -> +BATT
- J4 pad 38: I2C1_SDA -> SPI0_MOSI
- J4 pad 39: Net-(J4-Pad39) -> GND
- J4 pad 4: +3V3 -> +5V
- J4 pad 40: I2C1_SCL -> SPI0_MISO
- J4 pad 5: +5V -> I2C1_SCL
- J4 pad 6: +3.3VA -> GND
- J4 pad 7: GPIO16 -> +3.3VA
- J4 pad 8: GND -> UART0_TX
- J4 pad 9: GPIO17 -> GND
- R2 pad 1: EN -> Net-(R2-Pad1)
- U1 pad 3: EN -> Net-(R2-Pad1)
- U1 pad 5: +3V3 -> Net-(C2-Pad1)
Routing:
- net EN: track 51.2 -> 0.00 mm, vias 1 -> 0
- net +5V: track 106.7 -> 63.2 mm, vias 4 -> 2
- net Net-(J3-PadA4): track 0.00 -> 42.3 mm, vias 0 -> 2
- net +BATT: track 80.7 -> 40.2 mm, vias 1 -> 0
- net I2C1_SCL: track 18.9 -> 59.0 mm
- net I2C1_SDA: track 25.4 -> 63.8 mm
- net UART0_TX: track 41.3 -> 68.3 mm
- net UART0_RX: track 36.2 -> 61.6 mm
- net RESET: track 65.7 -> 49.5 mm
- net ADC3: track 39.4 -> 24.4 mm, vias 0 -> 1
- net LED2_BUILT_IN: track 51.2 -> 36.8 mm
- net +3.3VA: track 51.2 -> 37.1 mm, vias 2 -> 1
- net GPIO17: track 28.5 -> 15.4 mm, vias 1 -> 0
- net GPIO18: track 26.7 -> 14.4 mm
- net SDIO_DAT3: track 81.1 -> 69.4 mm
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Other:
- board text added: "+"
- board text added: "-"
- board text added: "3V"
- board text added: "v1.1"
- board text removed: "v1.0"

Commit message: microbyte-rp2040-v1.1 released
Parts:
- added G***: LOGO, LOGO:microbyte_new_font, B.Cu at (137.1, 101.7)
- added G***: LOGO, LOGO:microbyte_new_logo, B.Cu at (137.1, 92.8)
Routing:
- net GND: vias 65 -> 55
